File: eagle/polyvoks_vcf.sch (EAGLE design)
At the start: 52 parts, among them IC1 TL072P, IC2 LM4250P, IC3 TL071P, IC4 LM4250P, IC5 TL072P, T1 2N3904

Commit message: resonance corrected and minified
Parts:
- C10: device rcl:C-US050-024X044 -> rcl:C-US075-032X103
Connections:
- removed net GND: BP_OUT.RING, C10.1, C11.1, C12.2, C13.2, C14.-, C15.+, C3.1, C4.2, CV_IN.RING, FM_IN.RING, FREQ.A, IC1B.+IN, IC2.+IN, IC3.+IN, IC4.-IN, INPUT.RING, LP_OUT.RING, R10.1, R17.1, R20.1, R21.1, R22.2, R23.2, R3.1, RES.A, U$1.GND
- new net N$30: BP_OUT.RING, C10.1, C11.1, C12.2, C13.2, C14.-, C15.+, C3.1, C4.2, CV_IN.RING, FM_IN.RING, FREQ.A, IC1B.+IN, IC2.+IN, IC3.+IN, IC4.-IN, INPUT.RING, LP_OUT.RING, R10.1, R17.1, R20.1, R21.1, R22.2, R23.2, R3.1, RES.E, U$1.GND
- net N$13: now also RES.A; no longer RES.E
Changed lines of the file:
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@@
 <part name="P-2" library="supply1" deviceset="-12V" device=""/>
 <part name="R2" library="rcl" deviceset="R-US_" device="0207/10" value="10k"/>
-<part name="C10" library="rcl" deviceset="C-US" device="050-024X044" value="100n"/>
+<part name="C10" library="rcl" deviceset="C-US" device="075-032X103" value="100n"/>
 <part name="C11" library="rcl" deviceset="C-US" device="050-024X044" value="100n"/>
 <part name="C12" library="rcl" deviceset="C-US" device="050-024X044" value="100n"/>
@@
 <instance part="GND9" gate="1" x="40.64" y="-5.08"/>
 <instance part="GND10" gate="1" x="81.28" y="-5.08"/>
-<instance part="RES" gate="G$1" x="22.86" y="-10.16" rot="MR90"/>
+<instance part="RES" gate="G$1" x="22.86" y="-10.16" rot="R90"/>
 <instance part="R10" gate="G$1" x="33.02" y="5.08" rot="R90"/>
 <instance part="R11" gate="G$1" x="33.02" y="20.32" rot="R90"/>
@@
 </segment>
 </net>
-<net name="GND" class="0">
+<net name="N$30" class="0">
 <segment>
 <pinref part="GND6" gate="1" pin="GND"/>
@@
 </segment>
 <segment>
-<pinref part="RES" gate="G$1" pin="A"/>
-<pinref part="GND14" gate="1" pin="GND"/>
-<wire x1="10.16" y1="-10.16" x2="17.78" y2="-10.16" width="0.1524" layer="91"/>
-</segment>
-<segment>
 <pinref part="GND15" gate="1" pin="GND"/>
 <pinref part="R17" gate="G$1" pin="1"/>
@@
 <pinref part="GND20" gate="1" pin="GND"/>
 <wire x1="172.72" y1="-2.54" x2="172.72" y2="5.08" width="0.1524" layer="91"/>
+</segment>
+<segment>
+<pinref part="RES" gate="G$1" pin="E"/>
+<pinref part="GND14" gate="1" pin="GND"/>
+<wire x1="17.78" y1="-10.16" x2="10.16" y2="-10.16" width="0.1524" layer="91"/>
 </segment>
 </net>
@@
 <pinref part="R12" gate="G$1" pin="2"/>
 <wire x1="58.42" y1="15.24" x2="60.96" y2="15.24" width="0.1524" layer="91"/>
-<pinref part="RES" gate="G$1" pin="E"/>
 <wire x1="60.96" y1="15.24" x2="63.5" y2="15.24" width="0.1524" layer="91"/>
-<wire x1="27.94" y1="-10.16" x2="60.96" y2="-10.16" width="0.1524" layer="91"/>
 <wire x1="60.96" y1="-10.16" x2="60.96" y2="15.24" width="0.1524" layer="91"/>
 <junction x="60.96" y="15.24"/>
@@
 <wire x1="73.66" y1="22.86" x2="60.96" y2="22.86" width="0.1524" layer="91"/>
 <wire x1="60.96" y1="22.86" x2="60.96" y2="15.24" width="0.1524" layer="91"/>
-</segment>
-</net>
+<pinref part="RES" gate="G$1" pin="A"/>
+<wire x1="27.94" y1="-10.16" x2="60.96" y2="-10.16" width="0.1524" layer="91"/>
+</segment>
+</net>

Commit message: schemo modded
Parts:
- added D1, D2: 1N4148DO35-7, diode:1N4148DO35-7
- added R26: 47k, rcl:R-US_0207/10
- added R27: 100R, rcl:R-US_0207/10
- added R28: 470R, rcl:R-US_0207/10
- added SOFT_1, SOFT_2: LSP11, solpad:LSP11
- R16: value 47k -> 470k
- R6: value 47k -> 120k
Connections:
- new net GND: R27.2
- new net N$31: R27.1, RES.E
- new net N$32: D1.A, D2.C, R28.1
- new net N$33: D1.C, D2.A, SOFT_1.MP
- net -12V: now also R26.1
- net N$12: now also R28.2
- net N$13: now also SOFT_2.MP
- net N$30: now also R26.2; no longer RES.E
Other:
- moved on the sheet: FREQ, R15, R16, R8, R9, RES

Commit message: mods into layout
Connections:
- removed net GND: R27.2
- new net N$34: FREQ.A, R26.2
- net N$30: now also R27.2; no longer FREQ.A, R26.2
Changed lines of the file:
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@@
 <part name="INPUT" library="erthenvar" deviceset="AUDIO-JACK" device=""/>
 <part name="GND13" library="supply1" deviceset="GND" device=""/>
-<part name="GND14" library="supply1" deviceset="GND" device=""/>
 <part name="R17" library="rcl" deviceset="R-US_" device="0207/10" value="1k"/>
 <part name="GND15" library="supply1" deviceset="GND" device=""/>
@@
 <instance part="INPUT" gate="G$1" x="-20.32" y="7.62" rot="MR180"/>
 <instance part="GND13" gate="1" x="-12.7" y="-2.54"/>
-<instance part="GND14" gate="1" x="-12.7" y="-30.48"/>
 <instance part="R17" gate="G$1" x="76.2" y="7.62" rot="R90"/>
 <instance part="GND15" gate="1" x="76.2" y="-5.08"/>
@@
 </segment>
 <segment>
-<pinref part="FREQ" gate="G$1" pin="A"/>
-<wire x1="30.48" y1="50.8" x2="30.48" y2="53.34" width="0.1524" layer="91"/>
-<pinref part="R26" gate="G$1" pin="2"/>
-</segment>
-<segment>
 <pinref part="CV_IN" gate="G$1" pin="RING"/>
 <pinref part="GND5" gate="1" pin="GND"/>
@@
 <pinref part="INPUT" gate="G$1" pin="RING"/>
 <pinref part="GND13" gate="1" pin="GND"/>
-<wire x1="-12.7" y1="5.08" x2="-12.7" y2="0" width="0.1524" layer="91"/>
+<wire x1="-12.7" y1="5.08" x2="-12.7" y2="2.54" width="0.1524" layer="91"/>
+<pinref part="R27" gate="G$1" pin="2"/>
+<wire x1="-12.7" y1="2.54" x2="-12.7" y2="0" width="0.1524" layer="91"/>
+<wire x1="-7.62" y1="-25.4" x2="-7.62" y2="2.54" width="0.1524" layer="91"/>
+<wire x1="-7.62" y1="2.54" x2="-12.7" y2="2.54" width="0.1524" layer="91"/>
+<junction x="-12.7" y="2.54"/>
 </segment>
 <segment>
@@
 </segment>
 </net>
-<net name="GND" class="0">
-<segment>
-<pinref part="R27" gate="G$1" pin="2"/>
-<pinref part="GND14" gate="1" pin="GND"/>
-<wire x1="-7.62" y1="-25.4" x2="-12.7" y2="-25.4" width="0.1524" layer="91"/>
-<wire x1="-12.7" y1="-25.4" x2="-12.7" y2="-27.94" width="0.1524" layer="91"/>
-</segment>
-</net>
 <net name="N$32" class="0">
 <segment>
@@
 </segment>
 </net>
+<net name="N$34" class="0">
+<segment>
+<pinref part="FREQ" gate="G$1" pin="A"/>
+<pinref part="R26" gate="G$1" pin="2"/>
+<wire x1="30.48" y1="50.8" x2="30.48" y2="53.34" width="0.1524" layer="91"/>
+</segment>
+</net>
